File: kicad/Eve.kicad_sch (KiCad schematic)
At the start: 21 parts, among them J1 USB_C_Receptacle_USB2.0, SW1 SW_Push, U1 ATmega32U4-A, Y1 16MHz

Commit message: Add labels
Other:
- note added: "Decoupling Capacitors"
- note added: "MCU"
- note added: "Note: Place these as close to the I/C on PCB as you can"
- note added: "USB Port"
- moved on the sheet: C3, C4, C5, C7
